Commit message: add transmissions, add foot links, remove collisions

File: models/mini_cheetah/mini_cheetah_mesh.urdf (robot description, URDF)
Before this commit: robot mini_cheetah, 13 links, 12 joints
Links:
- added link LF_FOOT; collision sphere radius=0.0175; visual sphere radius=0.0175
- added link LH_FOOT; collision sphere radius=0.0175; visual sphere radius=0.0175
- added link RF_FOOT; collision sphere radius=0.0175; visual sphere radius=0.0175
- added link RH_FOOT; collision sphere radius=0.0175; visual sphere radius=0.0175
- link abduct_fl: geometry visual mesh filename=meshes/mini_abad.obj
- link abduct_fr: geometry visual mesh filename=meshes/mini_abad.obj
- link abduct_hl: geometry visual mesh filename=meshes/mini_abad.obj
- link abduct_hr: geometry visual mesh filename=meshes/mini_abad.obj
- link body: geometry visual mesh filename=meshes/mini_body.obj
- link shank_fl: geometry visual cylinder length=0.19 radius=0.015
- link shank_fr: geometry visual cylinder length=0.19 radius=0.015
- link shank_hl: geometry visual cylinder length=0.19 radius=0.015
- link shank_hr: geometry visual cylinder length=0.19 radius=0.015
- link thigh_fl: geometry visual mesh filename=meshes/mini_upper_link.obj
- link thigh_fr: geometry visual mesh filename=meshes/mini_upper_link.obj
- link thigh_hl: geometry visual mesh filename=meshes/mini_upper_link.obj
- link thigh_hr: geometry visual mesh filename=meshes/mini_upper_link.obj
Joints:
- added joint shank_fl_to_foot_fl: type fixed, parent shank_fl, child LF_FOOT, origin xyz=0.0 0.0 -0.195 rpy=0.0 0.0 0.0
- added joint shank_fr_to_foot_fr: type fixed, parent shank_fr, child RF_FOOT, origin xyz=0.0 0.0 -0.195 rpy=0.0 0.0 0.0
- added joint shank_hl_to_foot_hl: type fixed, parent shank_hl, child LH_FOOT, origin xyz=0.0 0.0 -0.195 rpy=0.0 0.0 0.0
- added joint shank_hr_to_foot_hr: type fixed, parent shank_hr, child RH_FOOT, origin xyz=0.0 0.0 -0.195 rpy=0.0 0.0 0.0

Commit message: misc urdf tweaks

File: models/mini_cheetah/mini_cheetah_mesh.urdf (robot description, URDF)
Before this commit: robot mini_cheetah, 17 links, 16 joints
Links:
- link body: geometry collision box size=0.23 0.19 0.1; visual mesh filename=meshes/mini_body.obj
- link shank_fl: geometry visual cylinder length=0.19 radius=0.010
- link shank_fr: geometry visual cylinder length=0.19 radius=0.010
- link shank_hl: geometry visual cylinder length=0.19 radius=0.010
- link shank_hr: geometry visual cylinder length=0.19 radius=0.010

File: models/mini_cheetah/mini_cheetah_simple_v2.urdf (robot description, URDF)
Before this commit: robot mini_cheetah, 17 links, 16 joints
Links:
- removed link foot_fl
- removed link foot_fr
- removed link foot_hl
- removed link foot_hr
- added link LF_FOOT; collision sphere radius=0.0175; visual sphere radius=0.0175
- added link LH_FOOT; collision sphere radius=0.0175; visual sphere radius=0.0175
- added link RF_FOOT; collision sphere radius=0.0175; visual sphere radius=0.0175
- added link RH_FOOT; collision sphere radius=0.0175; visual sphere radius=0.0175
Joints:
- removed joint fixed_shank_to_foot
- removed joint fixed_shank_to_foot_fr
- removed joint fixed_shank_to_foot_hl
- removed joint fixed_shank_to_foot_hr
- added joint shank_fl_to_foot_fl: type fixed, parent shank_fl, child LF_FOOT, origin xyz=0.0 0.0 -0.195 rpy=0.0 0.0 0.0
- added joint shank_fr_to_foot_fr: type fixed, parent shank_fr, child RF_FOOT, origin xyz=0.0 0.0 -0.195 rpy=0.0 0.0 0.0
- added joint shank_hl_to_foot_hl: type fixed, parent shank_hl, child LH_FOOT, origin xyz=0.0 0.0 -0.195 rpy=0.0 0.0 0.0
- added joint shank_hr_to_foot_hr: type fixed, parent shank_hr, child RH_FOOT, origin xyz=0.0 0.0 -0.195 rpy=0.0 0.0 0.0

Commit message: fix lower link mesh issues for mini cheetah

File: models/mini_cheetah/mini_cheetah_mesh.urdf (robot description, URDF)
Before this commit: robot mini_cheetah, 17 links, 16 joints
Links:
- link shank_fl: geometry visual mesh filename=meshes/mini_lower_link_.stl
- link shank_fr: geometry visual mesh filename=meshes/mini_lower_link_.stl
- link shank_hl: geometry visual mesh filename=meshes/mini_lower_link_.stl
- link shank_hr: geometry visual mesh filename=meshes/mini_lower_link_.stl
Joints:
- joint shank_fl_to_foot_fl: origin xyz=0.0 0.0 -0.195 rpy=0.0 0.0 0.0 -> xyz=0.0 0.0 -0.190 rpy=0.0 0.0 0.0
- joint shank_fr_to_foot_fr: origin xyz=0.0 0.0 -0.195 rpy=0.0 0.0 0.0 -> xyz=0.0 0.0 -0.190 rpy=0.0 0.0 0.0
- joint shank_hl_to_foot_hl: origin xyz=0.0 0.0 -0.195 rpy=0.0 0.0 0.0 -> xyz=0.0 0.0 -0.190 rpy=0.0 0.0 0.0
- joint shank_hr_to_foot_hr: origin xyz=0.0 0.0 -0.195 rpy=0.0 0.0 0.0 -> xyz=0.0 0.0 -0.190 rpy=0.0 0.0 0.0
